File: genesisctl.sch (KiCad schematic (older format))
At the start: 12 parts, among them J1 Conn_02x05_Odd_Even, J2 Screw_Terminal_01x02, J3 Screw_Terminal_01x04, J4 Screw_Terminal_01x04, U1 NE555, U2 74LS374, U3 74LS74, U4 74LS374

Commit message: added gerber files
Parts:
- C1, C2: value 3.3uF -> 0.22uF
Changed lines of the file:
@@
 P 1700 2600
 F 0 "C1" H 1815 2646 50  0000 L CNN
-F 1 "3.3uF" H 1815 2555 50  0000 L CNN
+F 1 "0.22uF" H 1815 2555 50  0000 L CNN
 F 2 "Capacitor_THT:CP_Radial_Tantal_D4.5mm_P5.00mm" H 1738 2450 50  0001 C CNN
 F 3 "~" H 1700 2600 50  0001 C CNN
@@
 P 3250 2600
 F 0 "C2" H 3365 2646 50  0000 L CNN
-F 1 "3.3uF" H 3365 2555 50  0000 L CNN
+F 1 "0.22uF" H 3365 2555 50  0000 L CNN
 F 2 "Capacitor_THT:CP_Radial_Tantal_D4.5mm_P5.00mm" H 3288 2450 50  0001 C CNN
 F 3 "~" H 3250 2600 50  0001 C CNN

Commit message: fixed reversed left/right
Connections:
- net btna_btnb: now also U4.3 (D0); no longer U4.7 (D2)
- net btna_out: now also J4.4 (Pin_4), U4.5 (O1); no longer J4.1 (Pin_1), U4.6 (O2)
- net gnd_left: now also U2.13 (D4); no longer U4.4 (D1)
- net gnd_right: now also U2.14 (D5); no longer U4.3 (D0)
- net left_out: now also U2.12 (O4); no longer U4.5 (O1)
- net right_out: now also U2.15 (O5); no longer U4.2 (O0)
- net start_btnc: now also U4.4 (D1); no longer U4.8 (D3)
- net start_out: no longer names the net of U4.9 (O3)
- net start_out: no longer J4.4 (Pin_4)
- new net: J4.1 (Pin_1), U4.2 (O0)
Changed lines of the file:
@@
 Wire Wire Line
 	4350 4300 3500 4300
-Wire Wire Line
-	3500 4300 3500 5000
 Text Label 3550 4300 0    50   ~ 0
 gnd_right
@@
 	4850 4300 5900 4300
 Wire Wire Line
-	5900 4300 5900 5300
+	5900 4300 5900 5100
 Text Label 5250 4100 0    50   ~ 0
 select
@@
 NoConn ~ 2950 5300
 NoConn ~ 1950 5300
-Text Label 7550 4800 1    50   ~ 0
-left_out
-Text Label 7650 4800 1    50   ~ 0
-right_out
 Text Label 8050 5100 1    50   ~ 0
 start_out
@@
 NoConn ~ 1950 5000
 Wire Wire Line
-	7750 4650 7750 5200
+	7750 4650 7750 5000
 Wire Wire Line
 	7450 4350 7450 4650
@@
 	3300 4650 7450 4650
 Wire Wire Line
-	6350 5200 6000 5200
-Wire Wire Line
-	7350 5200 7750 5200
-Wire Wire Line
-	6000 4000 6000 5200
-Connection ~ 6000 5200
+	6000 4000 6000 5000
 NoConn ~ 6350 5700
 NoConn ~ 7350 5700
-Wire Wire Line
-	7350 5300 8050 5300
-Wire Wire Line
-	8050 5300 8050 4650
-Wire Wire Line
-	6350 5300 5900 5300
-Connection ~ 5900 5300
 NoConn ~ 6350 5500
 NoConn ~ 7350 5500
@@
 	5600 1350 5600 2050
 Wire Wire Line
-	6000 5200 6000 5700
-Wire Wire Line
 	6000 5700 2950 5700
-NoConn ~ 2950 5400
-NoConn ~ 1950 5400
 Wire Wire Line
 	5900 5600 2950 5600
 Wire Wire Line
-	5900 5300 5900 5600
-NoConn ~ 2950 5500
-NoConn ~ 1950 5500
-Wire Wire Line
-	3500 5000 6350 5000
-Wire Wire Line
-	3400 5100 6350 5100
-Wire Wire Line
-	3400 4200 3400 5100
-Wire Wire Line
-	7550 5100 7350 5100
-Wire Wire Line
-	7550 4350 7550 5100
-Wire Wire Line
-	7350 5000 7650 5000
-Wire Wire Line
-	7650 5000 7650 4350
+	3400 5400 2950 5400
+Wire Wire Line
+	3500 5500 2950 5500
+Wire Wire Line
+	3400 4200 3400 5400
+Wire Wire Line
+	3500 4300 3500 5500
+Text GLabel 1950 5400 0    50   Output ~ 0
+left_out
+Text GLabel 7550 4350 3    50   Input ~ 0
+left_out
+Text GLabel 1950 5500 0    50   Output ~ 0
+right_out
+Text GLabel 7650 4350 3    50   Input ~ 0
+right_out
+Wire Wire Line
+	6000 5000 6350 5000
+Connection ~ 6000 5000
+Wire Wire Line
+	7350 5000 7750 5000
+Wire Wire Line
+	6000 5000 6000 5700
+NoConn ~ 6350 5200
+NoConn ~ 7350 5200
+Wire Wire Line
+	5900 5100 6350 5100
+Connection ~ 5900 5100
+Wire Wire Line
+	7350 5100 8050 5100
+Wire Wire Line
+	8050 5100 8050 4650
+Wire Wire Line
+	5900 5100 5900 5600
+NoConn ~ 7350 5300
+NoConn ~ 6350 5300
 $EndSCHEMATC
